Commit message: changed somethings

File: urdf/my_robot.urdf (robot description, URDF)
Before this commit: robot my_first_robot, 5 links, 4 joints
Joints:
- removed joint leftwheel_base
- added joint left_wheel_base: type continuous, parent base_link, child left_wheel, origin xyz=-0.25 -0.32 -0.25, axis 0.0 1.0 0.0

Commit message: added the differential drive custom dirve package

File: urdf/my_robot.urdf (robot description, URDF)
Before this commit: robot my_first_robot, 5 links, 4 joints
Links:
- link base_link: mass 10.0 -> 100.0

Commit message: remoed the my_world.sdf and also removed the sensors from the urdf

File: urdf/my_robot.urdf (robot description, URDF)
Before this commit: robot my_first_robot, 5 links, 4 joints
Joints:
- joint castorwheel_base_link: origin xyz=0.25 0 -0.35 -> xyz=-0.25 0 -0.35
- joint left_wheel_base: limit (none) -> effort=1000.0 velocity=20.0; origin xyz=-0.25 -0.32 -0.25 -> xyz=0.25 -0.32 -0.25
- joint right_wheel_base: limit (none) -> effort=1000.0 velocity=20.0; origin xyz=-0.25 0.32 -0.25 -> xyz=0.25 0.32 -0.25

Commit message: added te inertials tags and verified the working in gazebo

File: urdf/my_robot.urdf (robot description, URDF)
Before this commit: robot my_first_robot, 5 links, 4 joints
Links:
- link base_link: mass 100.0 -> 5.0
Joints:
- joint left_wheel_base: limit effort=1000.0 velocity=20.0 -> (none)
- joint right_wheel_base: limit effort=1000.0 velocity=20.0 -> (none)
