Commit message: successfully seted up the camera and the imu now going for the ekf fusion of the above two sensors

File: src/my_package/urdf/my_robot.urdf (robot description, URDF)
Before this commit: robot my_robot, 5 links, 4 joints
Links:
- added link camera_link, mass 0.1; collision box size=.03 .03 .03; visual box size=.03 .03 .03
- added link camera_optical
- added link imu_link
Joints:
- added joint base_camera: type fixed, parent base_link, child camera_link, origin xyz=0 0 .7 rpy=0 0.1745 0
- added joint base_imu: type fixed, parent base_link, child imu_link, origin xyz=0 0 0 rpy=0 0 0
- added joint camera_optical_camera: type fixed, parent camera_link, child camera_optical, origin xyz=0 0 0 rpy=-1.57 0 -1.57

Commit message: added the gps

File: src/my_package/urdf/my_robot.urdf (robot description, URDF)
Before this commit: robot my_robot, 8 links, 7 joints
Links:
- added link navsat_link
Joints:
- added joint base_navsat: type fixed, parent base_link, child navsat_link, origin xyz=0 0 0 rpy=0 0 0

Commit message: the robot now has all the required sensors and no ekf or other algorythms are done

File: src/my_package/urdf/my_robot.urdf (robot description, URDF)
Before this commit: robot my_robot, 9 links, 8 joints
Links:
- added link scan_link, mass 1e-5; collision box size=.1 .1 .1; visual box size=.1 .1 .1
Joints:
- added joint scan_joint: type fixed, parent base_link, child scan_link, origin xyz=0.0 0 0.25 rpy=0 0 0, axis 0 1 0
